Commit message: [260111] joing -> Joint, extension kit add

File: pointfoot/WF_TRON1A/xacro/leg.xacro (robot description, xacro)
@@ -3,5 +3,5 @@
     <xacro:include filename="$(find robot_description)/pointfoot/WF_TRON1A/xacro/transmission.xacro"/>
     <xacro:macro name="leg" params="name mirror mirror_STL *origin">
-        <joint name="abad_${name}_joint" type="revolute">
+        <joint name="abad_${name}_Joint" type="revolute">
             <origin
                 xyz="${abad_offset_x} ${abad_offset_y*mirror} ${abad_offset_z}"
@@ -35,5 +35,5 @@
             </inertial>
         </link>
-        <joint name="hip_${name}_joint" type="revolute">
+        <joint name="hip_${name}_Joint" type="revolute">
             <origin
                 xyz="${hip_offset_x} ${hip_offset_y*mirror} ${hip_offset_z}"
@@ -67,5 +67,5 @@
             </inertial>
         </link>
-        <joint name="knee_${name}_joint" type="revolute">
+        <joint name="knee_${name}_Joint" type="revolute">
             <origin
                 xyz="${knee_offset_x} ${knee_offset_y*mirror} ${knee_offset_z}"
@@ -105,5 +105,5 @@
             </inertial>
         </link>
-        <joint name="wheel_${name}_joint" type="revolute">
+        <joint name="wheel_${name}_Joint" type="revolute">
             <origin
                 xyz="${wheel_offset_x} ${wheel_offset_y*mirror} ${wheel_offset_z}"

File: pointfoot/WF_TRON1A/xacro/robot.xacro (robot description, xacro)
@@ -47,4 +47,7 @@
         <origin rpy="0 0 0" xyz="0 0 0"/>
     </joint>
+    <gazebo reference="imu_Joint">
+        <disableFixedJointLumping>true</disableFixedJointLumping>
+    </gazebo>
     <link name="imu_Link">
         <inertial>
@@ -101,28 +104,10 @@
     </xacro:leg>
    <xacro:if value="$(arg use_gazebo)">
-        <ros2_control name="pointfoot_gazebo_ros2_control_settings" type="system">
-            <hardware>
-                <plugin>pointfoot_gazebo/PointFootHWSim</plugin>
-            </hardware>
-            <xacro:leg_ros2_control_interface leg_name="L"/>
-            <xacro:leg_ros2_control_interface leg_name="R"/>
-            <sensor name="imu_sensor">
-                <frame_id name="imu_Link"/>
-                <state_interface name="orientation.x"/>
-                <state_interface name="orientation.y"/>
-                <state_interface name="orientation.z"/>
-                <state_interface name="orientation.w"/>
-                <state_interface name="angular_velocity.x"/>
-                <state_interface name="angular_velocity.y"/>
-                <state_interface name="angular_velocity.z"/>
-                <state_interface name="linear_acceleration.x"/>
-                <state_interface name="linear_acceleration.y"/>
-                <state_interface name="linear_acceleration.z"/>
-            </sensor>
-        </ros2_control>
+        <!-- ROS1 ros_control plugin: drives gazebo controller_manager for PointFootHWSim -->
         <gazebo>
-            <plugin filename="libgazebo_ros2_control.so" name="gazebo_ros2_control">
-                <robot_sim_type>pointfoot_gazebo/PointFootHWSim</robot_sim_type>
-                <parameters>$(find pointfoot_gazebo)/config/pointfoot_gazebo.yaml</parameters>
+            <plugin filename="libpointfoot_hw_sim.so" name="gazebo_ros_control">
+                <robotNamespace>/</robotNamespace>
+                <robotParam>robot_description</robotParam>
+                <robotSimType>pointfoot_gazebo/PointFootHWSim</robotSimType>
             </plugin>
         </gazebo>

File: pointfoot/WF_TRON1A/xacro/transmission.xacro (robot description, xacro)
@@ -2,40 +2,40 @@
 <robot xmlns:xacro="http://www.ros.org/wiki/xacro">
     <xacro:macro name="leg_transmission" params="name">
-        <transmission name="abad_${name}_joint_tran">
+        <transmission name="abad_${name}_Joint_tran">
             <type>transmission_interface/SimpleTransmission</type>
-            <joint name="abad_${name}_joint">
+            <joint name="abad_${name}_Joint">
             <hardwareInterface>hardware_interface/EffortJointInterface</hardwareInterface>
             </joint>
-            <actuator name="abad_${name}_joint_motor">
+            <actuator name="abad_${name}_Joint_motor">
             <hardwareInterface>hardware_interface/EffortJointInterface</hardwareInterface>
             <mechanicalReduction>1</mechanicalReduction>
             </actuator>
         </transmission>
-        <transmission name="hip_${name}_joint_tran">
+        <transmission name="hip_${name}_Joint_tran">
             <type>transmission_interface/SimpleTransmission</type>
-            <joint name="hip_${name}_joint">
+            <joint name="hip_${name}_Joint">
             <hardwareInterface>hardware_interface/EffortJointInterface</hardwareInterface>
             </joint>
-            <actuator name="hip_${name}_joint_motor">
+            <actuator name="hip_${name}_Joint_motor">
             <hardwareInterface>hardware_interface/EffortJointInterface</hardwareInterface>
             <mechanicalReduction>1</mechanicalReduction>
             </actuator>
         </transmission>
-        <transmission name="knee_${name}_joint_tran">
+        <transmission name="knee_${name}_Joint_tran">
             <type>transmission_interface/SimpleTransmission</type>
-            <joint name="knee_${name}_joint">
+            <joint name="knee_${name}_Joint">
             <hardwareInterface>hardware_interface/EffortJointInterface</hardwareInterface>
             </joint>
-            <actuator name="knee_${name}_joint_motor">
+            <actuator name="knee_${name}_Joint_motor">
             <hardwareInterface>hardware_interface/EffortJointInterface</hardwareInterface>
             <mechanicalReduction>1</mechanicalReduction>
             </actuator>
         </transmission>
-        <transmission name="wheel_${name}_joint_tran">
+        <transmission name="wheel_${name}_Joint_tran">
             <type>transmission_interface/SimpleTransmission</type>
-            <joint name="wheel_${name}_joint">
+            <joint name="wheel_${name}_Joint">
             <hardwareInterface>hardware_interface/EffortJointInterface</hardwareInterface>
             </joint>
-            <actuator name="wheel_${name}_joint_motor">
+            <actuator name="wheel_${name}_Joint_motor">
             <hardwareInterface>hardware_interface/EffortJointInterface</hardwareInterface>
             <mechanicalReduction>1</mechanicalReduction>
