Commit message: [260110]가제보에 센서키트 추가

File: pointfoot/WF_TRON1A/xacro/gazebo.xacro (robot description, xacro)
@@ -65,4 +65,42 @@
         <material>Gazebo/Red</material>
     </gazebo>
+    <!-- lidar extension kit  -->
+    <gazebo reference="mid360_link">
+        <sensor type="ray" name="laser_livox">
+        <pose>0 0 0 0 0 0</pose>
+        <visualize>true</visualize>
+        <always_on>true</always_on>
+        <update_rate>10</update_rate>
+        <plugin name="gazebo_ros_laser_controller" filename="liblivox_laser_simulation.so">
+            <ray>
+            <scan>
+                <horizontal>
+                <samples>100</samples>
+                <resolution>1</resolution>
+                <min_angle>-3.1415926535897931</min_angle>
+                <max_angle>3.1415926535897931</max_angle>
+                </horizontal>
+                <vertical>
+                <samples>50</samples>
+                <resolution>1</resolution>
+                <min_angle>-3.1415926535897931</min_angle>
+                <max_angle>3.1415926535897931</max_angle>
+                </vertical>
+            </scan>
+            <range>
+                <min>0.2</min>
+                <max>50</max>
+                <resolution>1</resolution>
+            </range>
+            </ray>
+            <samples>20000</samples>
+            <downsample>1</downsample>
+            <csv_file_name>mid360-real-centr.csv</csv_file_name>
+            <publish_pointcloud_type>2</publish_pointcloud_type>
+            <ros_topic>/livox/lidar</ros_topic>
+            <frameName>mid360_link</frameName>
+        </plugin>
+        </sensor>
+    </gazebo>
     <!-- Left leg -->
     <gazebo reference="abad_L_Link">

File: pointfoot/WF_TRON1A/xacro/robot.xacro (robot description, xacro)
@@ -67,4 +67,31 @@
         </collision>
     </link>
+    <!-- lidar extension kit  -->
+    <link name="extension_kit_link">
+        <visual>
+        <origin rpy="0 0 0" xyz="0 0 0"/>
+        <geometry>
+            <mesh filename="$(find robot_description)/pointfoot/WF_TRON1A/meshes/tron_extension_kit_assenbly.stl" scale="1 1 1"/>
+        </geometry>
+        </visual>
+    </link>
+    <joint name="extension_kit_joint" type="fixed">
+        <parent link="base_Link"/>
+        <child link="extension_kit_link"/>
+        <origin rpy="0 0 ${PI}" xyz="0 0 0.01"/>
+    </joint>
+    <link name="mid360_link">
+        <visual>
+        <origin rpy="0 0 0" xyz="0 0 0"/>
+        <geometry>
+            <mesh filename="$(find livox_laser_simulation)/meshes/livox_mid-360-90x.dae"/>
+        </geometry>
+        </visual>
+    </link>
+    <joint name="mid360_joint" type="fixed">
+        <parent link="extension_kit_link"/>
+        <child link="mid360_link"/>
+        <origin rpy="${PI} 0 0" xyz="0 0 0.182"/>
+    </joint>
     <xacro:leg name="L" mirror="1" mirror_STL="True">
         <origin rpy="0 0 0" xyz="0 0 0"/>

Commit message: [260122]expansion_mount추가

File: pointfoot/WF_TRON1A/xacro/gazebo.xacro (robot description, xacro)
@@ -36,5 +36,5 @@
     </gazebo> -->
     <!-- D435 Depth Camera (RealSense 토픽 호환) -->
-    <gazebo reference="d435_Link">
+    <gazebo reference="camera_link">
         <sensor name="d435_camera" type="depth">
             <update_rate>15</update_rate>
@@ -47,6 +47,6 @@
                 </image>
                 <clip>
-                    <near>0.2</near>
-                    <far>2.0</far>  <!-- clip_distance와 동일 -->
+                    <near>0.1</near>
+                    <far>10.0</far>
                 </clip>
             </camera>
@@ -61,4 +61,7 @@
                 <pointCloudTopicName>depth/color/points</pointCloudTopicName>
                 <frameName>camera_depth_optical_frame</frameName>
+                <!-- 포인트클라우드 거리 필터링 -->
+                <pointCloudCutoff>0.3</pointCloudCutoff>
+                <pointCloudCutoffMax>3.0</pointCloudCutoffMax>
             </plugin>
         </sensor>

File: pointfoot/WF_TRON1A/xacro/robot.xacro (robot description, xacro)
@@ -73,7 +73,7 @@
     <link name="extension_kit_link">
         <visual>
-        <origin rpy="0 0 ${PI}" xyz="0 0 0"/>
+        <origin rpy="0 0 0" xyz="0 0 0"/>
         <geometry>
-            <mesh filename="$(find robot_description)/pointfoot/WF_TRON1A/meshes/tron_extension_kit_assenbly.stl" scale="1 1 1"/>
+            <mesh filename="$(find robot_description)/pointfoot/WF_TRON1A/meshes/expansion_mount.stl" scale="1 1 1"/>
         </geometry>
         </visual>
@@ -82,5 +82,5 @@
         <parent link="base_Link"/>
         <child link="extension_kit_link"/>
-        <origin rpy="0 0 0" xyz="0 0 0.01"/>
+        <origin rpy="0 0 0" xyz="0 0 0.016"/>
     </joint>
     <link name="mid360_link">
@@ -95,12 +95,12 @@
         <parent link="extension_kit_link"/>
         <child link="mid360_link"/>
-        <origin rpy="${PI} 0 0" xyz="0 0 0.182"/>
+        <origin rpy="${PI} 0 0" xyz="0 0 0.162"/>
     </joint>
-    <!-- Livox IMU link (mid360_link와 동일 좌표계, 센서 분리용) -->
+    <!-- Livox IMU link (FAST-LIO extrinsic_T와 일치: LiDAR → IMU) -->
     <link name="livox_imu_link"/>
     <joint name="livox_imu_joint" type="fixed">
         <parent link="mid360_link"/>
         <child link="livox_imu_link"/>
-        <origin rpy="0 0 0" xyz="0 0 0"/>
+        <origin rpy="0 0 0" xyz="-0.011 -0.02329 0.04412"/>
     </joint>
     <xacro:leg name="L" mirror="1" mirror_STL="True">
@@ -121,11 +121,11 @@
     </xacro:if>
     <!-- ****************************************** extension kit D435 Camera ******************************************************** -->
-    <!-- 메인 카메라 링크 -->
-    <joint name="d435_joint" type="fixed">
-        <origin rpy="0 0.26179939 0" xyz="0.213 0 -0.017"/>
+    <!-- 카메라 링크 -->
+    <joint name="camera_joint" type="fixed">
+        <origin rpy="0 0.52359878 0" xyz="0.208 0 -0.0229"/>
         <parent link="base_Link"/>
-        <child link="d435_Link"/>
+        <child link="camera_link"/>
     </joint>
-    <link name="d435_Link">
+    <link name="camera_link">
         <visual>
             <origin rpy="1.5707963267948966 0 1.5707963267948966" xyz="0.0 0.0 0"/>
@@ -144,5 +144,5 @@
     <joint name="camera_depth_joint" type="fixed">
         <origin xyz="0 0 0" rpy="0 0 0"/>
-        <parent link="d435_Link"/>
+        <parent link="camera_link"/>
         <child link="camera_depth_frame"/>
     </joint>
@@ -158,5 +158,5 @@
     <joint name="camera_rgb_joint" type="fixed">
         <origin xyz="0 0 0" rpy="0 0 0"/>
-        <parent link="d435_Link"/>
+        <parent link="camera_link"/>
         <child link="camera_rgb_frame"/>
     </joint>

Commit message: [260123]camera0모델 추가

File: pointfoot/WF_TRON1A/xacro/gazebo.xacro (robot description, xacro)
@@ -35,5 +35,36 @@
         </plugin>
     </gazebo> -->
-    <!-- D435 Depth Camera (RealSense 토픽 호환) -->
+    <!-- camera0: 61도 아래 카메라 (elevation_mapping용) -->
+    <gazebo reference="camera0_link">
+        <sensor name="d435_camera0" type="depth">
+            <update_rate>15</update_rate>
+            <camera>
+                <horizontal_fov>1.047</horizontal_fov>
+                <image>
+                    <width>640</width>
+                    <height>480</height>
+                    <format>R8G8B8</format>
+                </image>
+                <clip>
+                    <near>0.1</near>
+                    <far>10.0</far>
+                </clip>
+            </camera>
+            <plugin name="d435_camera0_plugin" filename="libgazebo_ros_openni_kinect.so">
+                <alwaysOn>true</alwaysOn>
+                <updateRate>15.0</updateRate>
+                <cameraName>camera0</cameraName>
+                <imageTopicName>color/image_raw</imageTopicName>
+                <cameraInfoTopicName>color/camera_info</cameraInfoTopicName>
+                <depthImageTopicName>depth/image_rect_raw</depthImageTopicName>
+                <depthImageCameraInfoTopicName>depth/camera_info</depthImageCameraInfoTopicName>
+                <pointCloudTopicName>depth/color/points</pointCloudTopicName>
+                <frameName>camera0_depth_optical_frame</frameName>
+                <pointCloudCutoff>0.3</pointCloudCutoff>
+                <pointCloudCutoffMax>5.0</pointCloudCutoffMax>
+            </plugin>
+        </sensor>
+    </gazebo>
+    <!-- camera: 17도 아래 카메라 (사람 감지용) -->
     <gazebo reference="camera_link">
         <sensor name="d435_camera" type="depth">

File: pointfoot/WF_TRON1A/xacro/robot.xacro (robot description, xacro)
@@ -120,8 +120,56 @@
         </gazebo>
     </xacro:if>
-    <!-- ****************************************** extension kit D435 Camera ******************************************************** -->
-    <!-- 카메라 링크 -->
+    <!-- ****************************************** extension kit D435 Cameras ******************************************************** -->
+    <!-- camera0: 61도 아래 (elevation_mapping용) -->
+    <joint name="camera0_joint" type="fixed">
+        <origin rpy="0 1.063778179 0" xyz="0.13223 0.0222 -0.26826"/>
+        <parent link="base_Link"/>
+        <child link="camera0_link"/>
+    </joint>
+    <link name="camera0_link">
+        <visual>
+            <origin rpy="1.5707963267948966 0 1.5707963267948966" xyz="0.0 0.0 0"/>
+            <geometry>
+                <mesh filename="$(find robot_description)/pointfoot/meshes_camera/d435.dae"/>
+            </geometry>
+        </visual>
+        <collision>
+            <origin rpy="0 0 0" xyz="0 -0.0175 0"/>
+            <geometry>
+                <box size="0.02505 0.09 0.025"/>
+            </geometry>
+        </collision>
+    </link>
+    <!-- camera0 Depth Frame -->
+    <joint name="camera0_depth_joint" type="fixed">
+        <origin xyz="0 0 0" rpy="0 0 0"/>
+        <parent link="camera0_link"/>
+        <child link="camera0_depth_frame"/>
+    </joint>
+    <link name="camera0_depth_frame"/>
+    <!-- camera0 Depth Optical Frame (Z forward) -->
+    <joint name="camera0_depth_optical_joint" type="fixed">
+        <origin xyz="0 0 0" rpy="${-pi/2} 0 ${-pi/2}"/>
+        <parent link="camera0_depth_frame"/>
+        <child link="camera0_depth_optical_frame"/>
+    </joint>
+    <link name="camera0_depth_optical_frame"/>
+    <!-- camera0 RGB Frame -->
+    <joint name="camera0_rgb_joint" type="fixed">
+        <origin xyz="0 0 0" rpy="0 0 0"/>
+        <parent link="camera0_link"/>
+        <child link="camera0_rgb_frame"/>
+    </joint>
+    <link name="camera0_rgb_frame"/>
+    <!-- camera0 RGB Optical Frame (Z forward) -->
+    <joint name="camera0_rgb_optical_joint" type="fixed">
+        <origin xyz="0 0 0" rpy="${-pi/2} 0 ${-pi/2}"/>
+        <parent link="camera0_rgb_frame"/>
+        <child link="camera0_rgb_optical_frame"/>
+    </joint>
+    <link name="camera0_rgb_optical_frame"/>
+    <!-- camera: 17도 아래 (사람 감지용) -->
     <joint name="camera_joint" type="fixed">
-        <origin rpy="0 0.52359878 0" xyz="0.208 0 -0.0229"/>
+        <origin rpy="0 0.29670597 0" xyz="0.208 0 -0.0229"/>
         <parent link="base_Link"/>
         <child link="camera_link"/>
