Commit message: [260112]depth camera, 3d lidar 추가

File: pointfoot/PF_TRON1B/xacro/gazebo.xacro (robot description, xacro)
@@ -119,3 +119,35 @@
         <kd value="100.0"/>
     </gazebo>
+    <!-- ****************************************** D435 Depth Camera ******************************************************** -->
+    <gazebo reference="d435_Link">
+        <sensor name="d435_camera" type="depth">
+            <update_rate>15</update_rate>
+            <camera>
+                <horizontal_fov>1.047</horizontal_fov>
+                <image>
+                    <width>640</width>
+                    <height>480</height>
+                    <format>R8G8B8</format>
+                </image>
+                <clip>
+                    <near>0.1</near>
+                    <far>1.5</far>
+                </clip>
+            </camera>
+            <plugin name="d435_plugin" filename="libgazebo_ros_openni_kinect.so">
+                <alwaysOn>true</alwaysOn>
+                <updateRate>15.0</updateRate>
+                <cameraName>camera</cameraName>
+                <imageTopicName>color/image_raw</imageTopicName>
+                <cameraInfoTopicName>color/camera_info</cameraInfoTopicName>
+                <depthImageTopicName>depth/image_rect_raw</depthImageTopicName>
+                <depthImageCameraInfoTopicName>depth/camera_info</depthImageCameraInfoTopicName>
+                <pointCloudTopicName>depth/color/points</pointCloudTopicName>
+                <frameName>camera_depth_optical_frame</frameName>
+                <pointCloudCutoff>0.1</pointCloudCutoff>
+                <pointCloudCutoffMax>1.5</pointCloudCutoffMax>
+            </plugin>
+        </sensor>
+    </gazebo>
+    <!-- ****************************************** D435 Depth Camera END ******************************************************** -->
 </robot>

File: pointfoot/PF_TRON1B/xacro/robot.xacro (robot description, xacro)
@@ -102,5 +102,6 @@
     </xacro:if>
     <!-- ****************************************** D435 Camera ******************************************************** -->
-    <!-- <joint name="d435_joint" type="fixed">
+    <!-- 메인 카메라 링크 -->
+    <joint name="d435_joint" type="fixed">
         <origin rpy="0 1.063778179 0" xyz="0.13223 0.0222 -0.26826"/>
         <parent link="base_Link"/>
@@ -120,5 +121,33 @@
             </geometry>
         </collision>
-    </link> -->
+    </link>
+    <!-- Depth Frame -->
+    <joint name="camera_depth_joint" type="fixed">
+        <origin xyz="0 0 0" rpy="0 0 0"/>
+        <parent link="d435_Link"/>
+        <child link="camera_depth_frame"/>
+    </joint>
+    <link name="camera_depth_frame"/>
+    <!-- Depth Optical Frame (Z forward) -->
+    <joint name="camera_depth_optical_joint" type="fixed">
+        <origin xyz="0 0 0" rpy="${-pi/2} 0 ${-pi/2}"/>
+        <parent link="camera_depth_frame"/>
+        <child link="camera_depth_optical_frame"/>
+    </joint>
+    <link name="camera_depth_optical_frame"/>
+    <!-- RGB Frame -->
+    <joint name="camera_rgb_joint" type="fixed">
+        <origin xyz="0 0 0" rpy="0 0 0"/>
+        <parent link="d435_Link"/>
+        <child link="camera_rgb_frame"/>
+    </joint>
+    <link name="camera_rgb_frame"/>
+    <!-- RGB Optical Frame (Z forward) -->
+    <joint name="camera_rgb_optical_joint" type="fixed">
+        <origin xyz="0 0 0" rpy="${-pi/2} 0 ${-pi/2}"/>
+        <parent link="camera_rgb_frame"/>
+        <child link="camera_rgb_optical_frame"/>
+    </joint>
+    <link name="camera_rgb_optical_frame"/>
     <!-- ****************************************** D435 Camera END ******************************************************** -->
 </robot>

File: pointfoot/WF_TRON1A/xacro/gazebo.xacro (robot description, xacro)
@@ -35,4 +35,34 @@
         </plugin>
     </gazebo> -->
+    <!-- D435 Depth Camera (RealSense 토픽 호환) -->
+    <gazebo reference="d435_Link">
+        <sensor name="d435_camera" type="depth">
+            <update_rate>15</update_rate>
+            <camera>
+                <horizontal_fov>1.047</horizontal_fov>
+                <image>
+                    <width>640</width>
+                    <height>480</height>
+                    <format>R8G8B8</format>
+                </image>
+                <clip>
+                    <near>0.2</near>
+                    <far>2.0</far>  <!-- clip_distance와 동일 -->
+                </clip>
+            </camera>
+            <plugin name="d435_plugin" filename="libgazebo_ros_openni_kinect.so">
+                <alwaysOn>true</alwaysOn>
+                <updateRate>15.0</updateRate>
+                <cameraName>camera</cameraName>
+                <imageTopicName>color/image_raw</imageTopicName>
+                <cameraInfoTopicName>color/camera_info</cameraInfoTopicName>
+                <depthImageTopicName>depth/image_rect_raw</depthImageTopicName>
+                <depthImageCameraInfoTopicName>depth/camera_info</depthImageCameraInfoTopicName>
+                <pointCloudTopicName>depth/color/points</pointCloudTopicName>
+                <frameName>camera_depth_optical_frame</frameName>
+            </plugin>
+        </sensor>
+    </gazebo>
+    <!-- IMU sensor -->
     <gazebo reference="imu_Link">
         <gravity>true</gravity>
@@ -97,8 +127,29 @@
             <downsample>1</downsample>
             <csv_file_name>mid360-real-centr.csv</csv_file_name>
-            <publish_pointcloud_type>2</publish_pointcloud_type>
-            <ros_topic>/livox/lidar</ros_topic>
+            <publish_pointcloud_type>3</publish_pointcloud_type>
+            <ros_topic>/livox/lidar_sim</ros_topic>
             <frameName>mid360_link</frameName>
         </plugin>
+        </sensor>
+    </gazebo>
+    <!-- Livox Mid360 내장 IMU (시뮬레이션용) -->
+    <gazebo reference="livox_imu_link">
+        <gravity>true</gravity>
+        <sensor name="livox_imu_sensor" type="imu">
+            <always_on>true</always_on>
+            <update_rate>200</update_rate>
+            <visualize>false</visualize>
+            <topic>__default_topic__</topic>
+            <plugin filename="libgazebo_ros_imu_sensor.so" name="livox_imu_plugin">
+                <topicName>/livox/imu</topicName>
+                <bodyName>livox_imu_link</bodyName>
+                <updateRateHZ>200.0</updateRateHZ>
+                <gaussianNoise>0.0</gaussianNoise>
+                <xyzOffset>0 0 0</xyzOffset>
+                <rpyOffset>0 0 0</rpyOffset>
+                <frameName>livox_imu_link</frameName>
+                <initial_orientation_as_reference>false</initial_orientation_as_reference>
+            </plugin>
+            <pose>0 0 0 0 0 0</pose>
         </sensor>
     </gazebo>

File: pointfoot/WF_TRON1A/xacro/robot.xacro (robot description, xacro)
@@ -73,5 +73,5 @@
     <link name="extension_kit_link">
         <visual>
-        <origin rpy="0 0 0" xyz="0 0 0"/>
+        <origin rpy="0 0 ${PI}" xyz="0 0 0"/>
         <geometry>
             <mesh filename="$(find robot_description)/pointfoot/WF_TRON1A/meshes/tron_extension_kit_assenbly.stl" scale="1 1 1"/>
@@ -82,5 +82,5 @@
         <parent link="base_Link"/>
         <child link="extension_kit_link"/>
-        <origin rpy="0 0 ${PI}" xyz="0 0 0.01"/>
+        <origin rpy="0 0 0" xyz="0 0 0.01"/>
     </joint>
     <link name="mid360_link">
@@ -96,4 +96,11 @@
         <child link="mid360_link"/>
         <origin rpy="${PI} 0 0" xyz="0 0 0.182"/>
+    </joint>
+    <!-- Livox IMU link (mid360_link와 동일 좌표계, 센서 분리용) -->
+    <link name="livox_imu_link"/>
+    <joint name="livox_imu_joint" type="fixed">
+        <parent link="mid360_link"/>
+        <child link="livox_imu_link"/>
+        <origin rpy="0 0 0" xyz="0 0 0"/>
     </joint>
     <xacro:leg name="L" mirror="1" mirror_STL="True">
@@ -113,7 +120,8 @@
         </gazebo>
     </xacro:if>
-    <!-- ****************************************** D435 Camera ******************************************************** -->
-    <!-- <joint name="d435_joint" type="fixed">
-        <origin rpy="0 1.063778179 0" xyz="0.13223 0.0222 -0.26826"/>
+    <!-- ****************************************** extension kit D435 Camera ******************************************************** -->
+    <!-- 메인 카메라 링크 -->
+    <joint name="d435_joint" type="fixed">
+        <origin rpy="0 0.26179939 0" xyz="0.213 0 -0.017"/>
         <parent link="base_Link"/>
         <child link="d435_Link"/>
@@ -121,5 +129,5 @@
     <link name="d435_Link">
         <visual>
-            <origin rpy="1.5707963267948966 0 1.5707963267948966" xyz="0.0149 -0.0175 0"/>
+            <origin rpy="1.5707963267948966 0 1.5707963267948966" xyz="0.0 0.0 0"/>
             <geometry>
                 <mesh filename="$(find robot_description)/pointfoot/meshes_camera/d435.dae"/>
@@ -132,5 +140,33 @@
             </geometry>
         </collision>
-    </link> -->
+    </link>
+    <!-- Depth Frame -->
+    <joint name="camera_depth_joint" type="fixed">
+        <origin xyz="0 0 0" rpy="0 0 0"/>
+        <parent link="d435_Link"/>
+        <child link="camera_depth_frame"/>
+    </joint>
+    <link name="camera_depth_frame"/>
+    <!-- Depth Optical Frame (Z forward) -->
+    <joint name="camera_depth_optical_joint" type="fixed">
+        <origin xyz="0 0 0" rpy="${-pi/2} 0 ${-pi/2}"/>
+        <parent link="camera_depth_frame"/>
+        <child link="camera_depth_optical_frame"/>
+    </joint>
+    <link name="camera_depth_optical_frame"/>
+    <!-- RGB Frame -->
+    <joint name="camera_rgb_joint" type="fixed">
+        <origin xyz="0 0 0" rpy="0 0 0"/>
+        <parent link="d435_Link"/>
+        <child link="camera_rgb_frame"/>
+    </joint>
+    <link name="camera_rgb_frame"/>
+    <!-- RGB Optical Frame (Z forward) -->
+    <joint name="camera_rgb_optical_joint" type="fixed">
+        <origin xyz="0 0 0" rpy="${-pi/2} 0 ${-pi/2}"/>
+        <parent link="camera_rgb_frame"/>
+        <child link="camera_rgb_optical_frame"/>
+    </joint>
+    <link name="camera_rgb_optical_frame"/>
     <!-- ****************************************** D435 Camera END ******************************************************** -->
 </robot>

File: pointfoot/WF_TRON1B/xacro/gazebo.xacro (robot description, xacro)
@@ -97,8 +97,29 @@
             <downsample>1</downsample>
             <csv_file_name>mid360-real-centr.csv</csv_file_name>
-            <publish_pointcloud_type>2</publish_pointcloud_type>
-            <ros_topic>/livox/lidar</ros_topic>
+            <publish_pointcloud_type>3</publish_pointcloud_type>
+            <ros_topic>/livox/lidar_sim</ros_topic>
             <frameName>mid360_link</frameName>
         </plugin>
+        </sensor>
+    </gazebo>
+    <!-- Livox Mid360 내장 IMU (시뮬레이션용) -->
+    <gazebo reference="livox_imu_link">
+        <gravity>true</gravity>
+        <sensor name="livox_imu_sensor" type="imu">
+            <always_on>true</always_on>
+            <update_rate>200</update_rate>
+            <visualize>false</visualize>
+            <topic>__default_topic__</topic>
+            <plugin filename="libgazebo_ros_imu_sensor.so" name="livox_imu_plugin">
+                <topicName>/livox/imu</topicName>
+                <bodyName>livox_imu_link</bodyName>
+                <updateRateHZ>200.0</updateRateHZ>
+                <gaussianNoise>0.0</gaussianNoise>
+                <xyzOffset>0 0 0</xyzOffset>
+                <rpyOffset>0 0 0</rpyOffset>
+                <frameName>livox_imu_link</frameName>
+                <initial_orientation_as_reference>false</initial_orientation_as_reference>
+            </plugin>
+            <pose>0 0 0 0 0 0</pose>
         </sensor>
     </gazebo>

File: pointfoot/WF_TRON1B/xacro/robot.xacro (robot description, xacro)
@@ -86,5 +86,5 @@
     <link name="mid360_link">
         <visual>
-        <origin rpy="0 0 0" xyz="0 0 0"/>
+        <origin rpy="${PI} 0 0" xyz="0 0 0"/>
         <geometry>
             <mesh filename="$(find livox_laser_simulation)/meshes/livox_mid-360-90x.dae"/>
@@ -95,5 +95,12 @@
         <parent link="extension_kit_link"/>
         <child link="mid360_link"/>
-        <origin rpy="${PI} 0 0" xyz="0 0 0.182"/>
+        <origin rpy="0 0 0" xyz="0 0 0.182"/>
+    </joint>
+    <!-- Livox IMU link (mid360_link와 동일 좌표계, 센서 분리용) -->
+    <link name="livox_imu_link"/>
+    <joint name="livox_imu_joint" type="fixed">
+        <parent link="mid360_link"/>
+        <child link="livox_imu_link"/>
+        <origin rpy="0 0 0" xyz="0 0 0"/>
     </joint>
     <xacro:leg name="L" mirror="1" mirror_STL="True">
